File: hardware/led-adapter/neohex-passive-rev-a/kicad/neohex-passive-rev-a.kicad_pcb (KiCad board)
At the start: 2 copper layers, 60 x 35 mm, 18 parts, among them J1 GROVE_OUT_PH4_PLACEHOLDER, J2 VLED_IN, J3 STEMMA_DATA, J4 GPIO_DATA

Commit message: Add NeoHEX adapter PCBWay package
Parts:
- added J5: QT_GROVE_OUT, JST_SH_BM04B-SRSS-TB_1x04-1MP_P1.00mm_Vertical, F.Cu at (58.0, 29.0)
- J1: value GROVE_OUT_PH4_PLACEHOLDER -> HY2.0_4P_SMD_OUT; footprint JST_PH_B4B-PH-K_1x04_P2.00mm_Vertical -> M5Stack_HY2.0-4P_SMD_A118
- J2: footprint JST_PH_B2B-PH-K_1x02_P2.00mm_Vertical -> JST_PH_S2B-PH-SM4-TB_1x02-1MP_P2.00mm_Horizontal
- moved H2 12.0 mm to (68.0, 31.0)
- moved J1 9.00 mm to (64.0, 12.0), turned to 0 degrees
- moved J2 6.92 mm to (11.8, 7.00)
- moved TP5 3.61 mm to (52.0, 24.0)
Routing:
- net GND: track 141.1 -> 187.9 mm, vias 0 -> 2
- net DATA_OUT: track 11.1 -> 43.8 mm, vias 0 -> 2
- net NC_WHITE: track 8.00 -> 38.2 mm, vias 0 -> 2
- net VLED: track 89.6 -> 116.3 mm, vias 0 -> 2
Other:
- board size 60 x 35 mm -> 72 x 35 mm
- board text added: "J1 HY2.0 SMD"
- board text added: "J5 QT-GROVE OUT"
- board text removed: "J1 PH4 PLACEHOLDER"
