File: hardware/capboard/capbank_placement_4pin.kicad_pcb (KiCad board)
At the start: 2 copper layers, 100 x 40 mm, 31 parts, among them SW1 SW_Push_1TS009xxxx-xxxx-xxxx_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, U1 HT7550-1, U2 MT3608

Commit message: hardware/capboard: 4-pin variant silkscreen reads D7 VDC GND GND, recentred on the 4-pin span
Co-Authored-By: Claude Fable 5 <noreply@anthropic.com>
Claude-Session: https://claude.ai/code/session_01XEHUfVFPdvg3k1kXt9D9MK
Other:
- board text added: "D7 VDC GND GND"
- board text removed: "D7 VDC GND"
Changed lines of the file:
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@@
 		)
 	)
-	(gr_text "D7 VDC GND"
+	(gr_text "D7 VDC GND GND"
 		(at 13.5 27.5 0)
 		(layer "F.SilkS")
@@
 		)
 	)
-	(gr_text "D7 VDC GND"
+	(gr_text "D7 VDC GND GND"
 		(at 74 27.5 0)
 		(layer "F.SilkS")
